File: YuSynth_Metalizer/Hardware/YuSynth_Metalizer_main/YuSynth_Metalizer_main.kicad_pcb (KiCad board)
At the start: 2 copper layers, 29 x 109 mm, 83 parts, among them J37 CV1, J38 CV2, J39 In, J40 Out, J41 Conn_01x10, J42 Conn_01x10, J43 Conn_01x10, J44 Conn_01x10, J45 Conn_02x05_Odd_Even, Q1 BC547, Q10 BC547, Q11 BC557, Q12 BC547, Q2 BC547, Q3 BC547, Q4 BC547, Q5 BC557, Q6 BC547, Q7 BC557, Q8 BC547, Q9 BC557, U1 TL072, U2 TL074

Commit message: Redid all boards
Parts:
- removed C11: 10µ, Capacitor_THT:CP_Radial_D6.3mm_P2.50mm
- removed C41, C42: 47uf, Capacitor_THT:CP_Radial_D6.3mm_P2.50mm
- removed J37: CV1, Connector_Audio:Jack_3.5mm_QingPu_WQP-PJ398SM_Vertical_CircularHoles
- removed J38: CV2, Connector_Audio:Jack_3.5mm_QingPu_WQP-PJ398SM_Vertical_CircularHoles
- removed J39: In, Connector_Audio:Jack_3.5mm_QingPu_WQP-PJ398SM_Vertical_CircularHoles
- removed J40: Out, Connector_Audio:Jack_3.5mm_QingPu_WQP-PJ398SM_Vertical_CircularHoles
- removed J41, J42, J43, J44: Conn_01x10, Connector_PinHeader_2.54mm:PinHeader_1x10_P2.54mm_Vertical
- removed J45: Conn_02x05_Odd_Even, Connector_IDC:IDC-Header_2x05_P2.54mm_Vertical
- removed R12, R13, R44: 270k, Resistor_THT:R_Axial_DIN0207_L6.3mm_D2.5mm_P7.62mm_Horizontal
- removed RV37: CV1, Potentiometer_THT:Potentiometer_Alpha_RD901F-40-00D_Single_Vertical
- removed RV38: CV2, Potentiometer_THT:Potentiometer_Alpha_RD901F-40-00D_Single_Vertical
- removed RV39: Shape, Potentiometer_THT:Potentiometer_Alpha_RD901F-40-00D_Single_Vertical
- added J1: Conn_01x06, Connector_PinSocket_2.54mm:PinSocket_1x06_P2.54mm_Vertical, B.Cu at (12.7, 21.8)
- added J2: Conn_01x10, Connector_PinSocket_2.54mm:PinSocket_1x10_P2.54mm_Vertical, B.Cu at (12.7, 94.0)
- added J3: Conn_01x10, Connector_PinSocket_2.54mm:PinSocket_1x10_P2.54mm_Vertical, B.Cu at (-12.7, 94.0)
- added J4: Conn_01x06, Connector_PinSocket_2.54mm:PinSocket_1x06_P2.54mm_Vertical, B.Cu at (-12.7, 21.8)
- C37, C38, C39, C40: footprint Capacitor_THT:C_Rect_L7.0mm_W2.0mm_P5.00mm -> Capacitor_THT:C_Rect_L4.6mm_W2.0mm_P2.50mm_MKS02_FKP02
- R10, R11, R14, R15, R16, R17, R18, R19, R20, R21, R22, R23, R24, R25, R26, R27, R28, R29, R3, R30, R31, R32, R33, R34, R35, R36, R37, R38, R39, R4, R40, R41, R42, R43, R5, R6, R7, R8, R9: footprint Resistor_THT:R_Axial_DIN0207_L6.3mm_D2.5mm_P7.62mm_Horizontal -> Resistor_THT:R_Axial_DIN0204_L3.6mm_D1.6mm_P7.62mm_Horizontal
- moved C9 238.7 mm to (-9.91, 68.9)
- moved C39 233.9 mm to (-9.65, 40.3)
- moved C7 227.8 mm to (-9.91, 58.6)
- moved C3 226.4 mm to (9.40, 53.6)
- moved R19 221.3 mm to (6.10, 116.8)
- moved R20 221.3 mm to (6.10, 101.6)
- moved R26 221.3 mm to (6.10, 67.6)
- moved R27 221.3 mm to (6.10, 52.3)
- moved R21 220.8 mm to (3.56, 116.8)
- moved R24 220.8 mm to (3.56, 101.6)
- moved R28 220.8 mm to (3.56, 59.9)
- moved C37 220.5 mm to (-1.52, 91.4), turned to 0 degrees
- moved C40 220.4 mm to (-1.48, 77.7), turned to 0 degrees
- moved R22 220.3 mm to (1.02, 109.2)
- moved R23 220.3 mm to (1.02, 101.6)
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Connections:
- net Net-(C10-Pad2) renamed OUT
- net Net-(U1A--) renamed CV_IN
- R3 pad 1: Net-(J39-PadT) -> IN
Routing:
- net Net-(C3-Pad1): track 80.3 -> 34.2 mm
- net Net-(C9-Pad2): track 3.84 -> 46.4 mm
- net Net-(C3-Pad2): track 27.0 -> 60.7 mm
- net Net-(C8-Pad2): track 40.6 -> 13.8 mm
- net Net-(C5-Pad2): track 0.00 -> 20.3 mm
- net -12V: track 187.8 -> 169.4 mm, vias 1 -> 0
- net OUT: track 0.00 -> 16.0 mm
- net Net-(Q3-E): track 0.00 -> 15.0 mm
- net +12V: track 176.3 -> 161.4 mm, vias 0 -> 2
- net CV_IN: track 5.00 -> 18.9 mm
- net IN: track 0.00 -> 12.1 mm
- net Net-(U2A--): track 14.6 -> 3.57 mm
- net Net-(U2B--): track 14.5 -> 3.57 mm
- net Net-(Q1-B): track 4.27 -> 14.8 mm
- net Net-(R14-Pad2): track 4.49 -> 12.5 mm
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Other:
- board size 29 x 109 mm -> 29 x 98.7 mm
