File: YuSynth_Metalizer/Hardware/YuSynth_Metalizer_main/YuSynth_Metalizer_main.kicad_sch (KiCad schematic)
At the start: 83 parts, among them J37 CV1, J38 CV2, J39 In, J40 Out, J41 Conn_01x10, J42 Conn_01x10, J43 Conn_01x10, J44 Conn_01x10, J45 Conn_02x05_Odd_Even, Q1 BC547, Q10 BC547, Q11 BC557, Q12 BC547, Q2 BC547, Q3 BC547, Q4 BC547, Q5 BC557, Q6 BC547, Q7 BC557, Q8 BC547, Q9 BC557, U1 TL072, U2 TL074

Commit message: Redid all boards
Parts:
- removed C11: 10µ, Capacitor_THT:CP_Radial_D6.3mm_P2.50mm, symbol Device:C_Polarized
- removed C41, C42: 47uf, Capacitor_THT:CP_Radial_D6.3mm_P2.50mm, symbol Device:C_Polarized
- removed J37: CV1, Connector_Audio:Jack_3.5mm_QingPu_WQP-PJ398SM_Vertical_CircularHoles, symbol Connector:AudioJack2
- removed J38: CV2, Connector_Audio:Jack_3.5mm_QingPu_WQP-PJ398SM_Vertical_CircularHoles, symbol Connector:AudioJack2
- removed J39: In, Connector_Audio:Jack_3.5mm_QingPu_WQP-PJ398SM_Vertical_CircularHoles, symbol Connector:AudioJack2
- removed J40: Out, Connector_Audio:Jack_3.5mm_QingPu_WQP-PJ398SM_Vertical_CircularHoles, symbol Connector:AudioJack2
- removed J42, J43: Conn_01x10, Connector_PinHeader_2.54mm:PinHeader_1x10_P2.54mm_Vertical, symbol Connector_Generic:Conn_01x10
- removed J45: Conn_02x05_Odd_Even, Connector_IDC:IDC-Header_2x05_P2.54mm_Vertical, symbol Connector_Generic:Conn_02x05_Odd_Even
- removed R12, R13, R44: 270k, Resistor_THT:R_Axial_DIN0207_L6.3mm_D2.5mm_P7.62mm_Horizontal, symbol Device:R
- removed RV37: CV1, Potentiometer_THT:Potentiometer_Alpha_RD901F-40-00D_Single_Vertical, symbol Device:R_Potentiometer
- removed RV38: CV2, Potentiometer_THT:Potentiometer_Alpha_RD901F-40-00D_Single_Vertical, symbol Device:R_Potentiometer
- removed RV39: Shape, Potentiometer_THT:Potentiometer_Alpha_RD901F-40-00D_Single_Vertical, symbol Device:R_Potentiometer
- added J1, J4: Conn_01x06, Connector_PinSocket_2.54mm:PinSocket_1x06_P2.54mm_Vertical, symbol Connector_Generic:Conn_01x06
- C37, C38, C39, C40: footprint Capacitor_THT:C_Rect_L7.0mm_W2.0mm_P5.00mm -> Capacitor_THT:C_Rect_L4.6mm_W2.0mm_P2.50mm_MKS02_FKP02
- J2: renamed from J41; footprint Connector_PinHeader_2.54mm:PinHeader_1x10_P2.54mm_Vertical -> Connector_PinSocket_2.54mm:PinSocket_1x10_P2.54mm_Vertical
- J3: renamed from J44; footprint Connector_PinHeader_2.54mm:PinHeader_1x10_P2.54mm_Vertical -> Connector_PinSocket_2.54mm:PinSocket_1x10_P2.54mm_Vertical
- R10, R11, R14, R15, R16, R17, R18, R19, R20, R21, R22, R23, R24, R25, R26, R27, R28, R29, R3, R30, R31, R32, R33, R34, R35, R36, R37, R38, R39, R4, R40, R41, R42, R43, R5, R6, R7, R8, R9: footprint Resistor_THT:R_Axial_DIN0207_L6.3mm_D2.5mm_P7.62mm_Horizontal -> Resistor_THT:R_Axial_DIN0204_L3.6mm_D1.6mm_P7.62mm_Horizontal
Connections:
- net +12V: now also J2.9 (Pin_9), J3.1 (Pin_1), J3.9 (Pin_9), J4.6 (Pin_6)
- net -12V: now also J2.1 (Pin_1), J2.10 (Pin_10), J3.10 (Pin_10), J1.6 (Pin_6)
- net GND: now also J2.2 (Pin_2), J2.8 (Pin_8), J3.2 (Pin_2), J3.4 (Pin_4), J3.8 (Pin_8), J1.3 (Pin_3), J1.5 (Pin_5), J4.3 (Pin_3), J4.5 (Pin_5)
- net CV_IN: now reaches R14.1, U1.2 (-)
- net CV_IN: now also J4.4 (Pin_4)
- net OUT: now reaches J3.3 (Pin_3)
- net OUT: now also C10.2, R41.2, U2.1
- net IN: now reaches R3.1
- net IN: now also J1.4 (Pin_4)
Other:
- moved on the sheet: J3
