File: Xor-tillator/Hardware/Xor-tillator_main/Xor-tillator_main.kicad_sch (KiCad schematic)
At the start: 42 parts, among them J1 Tune CV In, J2 PowerConn, Q1 2N3904, U1 4070, U2 40106, U3 TL072, U4 4070, U5 TL072

Commit message: Continued with XOR-tillator
Parts:
- removed unit 3 of U3
- added C13: 100pf, symbol Device:C
- added C14, C16, C20: 1uf, symbol Device:C
- added C15, C17, C19, C21: 1200pf, symbol Device:C
- added C18: 10uf, symbol Device:C
- added R17, R18, R19, R20, R21, R30, R31, R32, R33, R35, R38: 100k, symbol Device:R
- added R22, R23, R24, R25, R26, R27, R28, R29: 680k?, symbol Device:R
- added R34, R37, R39: ?, symbol Device:R
- added R36: Mode Value?, symbol Device:R
- added R40: 5.1k, symbol Device:R
- added R41: 1k, symbol Device:R
- added R42, R44, R46, R48: 20k, symbol Device:R
- added R43, R45, R47, R49: 220R, symbol Device:R
- added RV10, RV11, RV12, RV13, RV14, RV15, RV16, RV9: 1M?, symbol Device:R_Potentiometer_Trim
- added RV_EXT1, RV_EXT2: 100k, symbol Device:R_Potentiometer
- added SW1: EXT_IN1_SW, symbol Switch:SW_SPDT
- added SW2: EXT_IN2_SW, symbol Switch:SW_SPDT
- added SW3: HOLD_A, symbol Switch:SW_SPDT_MSM
- added SW4: HOLD_Ext, symbol Switch:SW_SPDT_MSM
- added SW5: HOLD_B, symbol Switch:SW_SPDT_MSM
- added SW6: HOLD_C, symbol Switch:SW_SPDT_MSM
- added U10: TL072, symbol Amplifier_Operational:TL072
- added unit 3 of U4
- added unit 4 of U4
- added unit 1 of U4
- added unit 2 of U4
- added unit 2 of U5
- added unit 4 of U5
- added unit 3 of U5
- added U6: SSI2164, Package_SO:SOIC-16_3.9x9.9mm_P1.27mm, symbol Audio:SSI2164
- added U7: TL072, symbol Amplifier_Operational:TL074
- added U8, U9: 4070, symbol 4xxx:4070
- U4: now in the parts list
- U5: value TL072 -> TL074; symbol Amplifier_Operational:TL072 -> Amplifier_Operational:TL074
Connections:
- net +12V: now also R36.1, U6.16 (V+)
- net -12V: now also U6.9 (V-)
- net A: now also SW3.2 (3), U4.5, U8.2
- net AL: now also RV9.2, RV9.3
- net AR: now also RV10.2, RV10.3, SW2.3 (C)
- net B: now also SW5.2 (3), U4.6, U4.8
- net BL: now also RV13.2, RV13.3
- net BR: now also RV14.2, RV14.3
- net C: now also SW6.2 (3), U4.9
- net CL: now also RV15.2, RV15.3
- net CR: now also RV16.2, RV16.3
- net GND: now also C15.1, C17.1, C19.1, C21.1, RV_EXT1.3, RV_EXT2.3, U10.3 (+), U5.10 (+), U5.12 (+), U5.5 (+), U6.8 (GND), U7.3 (+), U7.5 (+)
- net at R13.2, R14.2, R15.2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: now also R21.2
- net OSC1: now reaches R2.2, U1.2, U2.4
- net OSC1: now also SW1.3 (C)
- net MIX1: now reaches R16.2, U5.1
- net MIX1: now also C14.1
- new net: C13.1, R40.1, U10.2 (-), U6.12 (I_OUT3), U6.13 (I_OUT4), U6.4 (I_OUT1), U6.5 (I_OUT2)
- new net: C13.2, R40.2, R41.1, U10.1
- new net: C20.2, R48.1
- new net: C19.2, R47.1
- new net: R30.2, R31.2, R32.2, R34.1, U5.6 (-)
- new net: C14.2, R42.1
- new net: C18.2, R46.1
- new net: C17.2, R45.1
- new net: R27.2, RV14.1
- new net: R33.2, R35.2, R37.1, U5.9 (-)
- new net: R19.2, R20.1, U7.6 (-)
- new net: R20.2, RV_EXT2.1, U7.7
- new net: R22.1, SW3.1
- new net: R23.1, SW3.3 (4)
- new net: C21.2, R49.1
- new net: R38.2, R39.1, U5.13 (-)
- new net: R18.2, RV_EXT1.1, U7.1
- new net: R17.2, R18.1, U7.2 (-)
- new net: R24.1, SW4.1
- new net: R25.1, SW4.3 (4)
- new net: R28.1, SW6.1
- new net: R28.2, RV15.1
- new net: R27.1, SW5.3 (4)
- new net: R24.2, RV11.1
- new net: RV_EXT2.2, SW2.1 (A)
- new net: SW2.2 (B), U4.2
- new net: RV_EXT1.2, SW1.1 (A)
- new net: R29.1, SW6.3 (4)
- new net: R36.2, U6.1 (MODE)
- new net: R25.2, RV12.1
- new net: R26.1, SW5.1
- new net: R26.2, RV13.1
- new net: R22.2, RV9.1
- new net: C16.2, R44.1
- new net: R29.2, RV16.1
- new net: R23.2, RV10.1
- new net: C15.2, R43.1
- new net AB: R31.1, U4.13, U4.4, U5.1
- new net AB_BC: R35.1, U5.3, U9.2
- new net BC: R32.1, U4.10, U5.2
- new net E: R21.1, SW4.2 (3), U8.1
- new net EA: R30.1, U4.12, U8.3
- new net EA_AB: R33.1, U4.11, U9.1
- new net EXT_IN1: R17.1
- new net EXT_IN2: R19.1
- new net ExtL: RV11.2, RV11.3, SW1.2 (B), U4.1
- new net ExtR: RV12.2, RV12.3, U4.3
- new net I_MIX1: R42.2, R43.2, U6.2 (I_IN1)
- new net I_MIX2: R44.2, R45.2, U6.7 (I_IN2)
- new net I_MIX3: R46.2, R47.2, U6.10 (I_IN3)
- new net I_MIX4: R48.2, R49.2, U6.15 (I_IN4)
- new net MIX2: C16.1, R34.2, U5.7
- new net MIX3: C18.1, R37.2, U5.8
- new net MIX4: C20.1, R39.2, U5.14
- new net XOR_SUM: R38.1, U9.3
Other:
- note added: "EXT. IN"
- note added: "HOLD SYSTEM"
- note added: "SECOND_XOR_STAGE"
- note added: "soll ich direkt von mixer widerständen (r13, r14 ,..) in den ssi2164 und mix1 - mix4 sind buchsen - ausgänge (mit 1k vorwiderstand) ?"
- moved on the sheet: R13, R14, R15, R16, U5A

Commit message: continued XOR-tillator
Parts:
- added C10, C11, C9: 100pf, symbol Device:C
- added R50, R52, R54: 5.1k, symbol Device:R
- added R51, R53, R55, R61: 1k, symbol Device:R
- added R56, R57, R58, R59, R60: 100k, symbol Device:R
- added unit 1 of U7
- added unit 3 of U7
- added unit 4 of U7
- added U8: TL072, symbol Amplifier_Operational:TL072
- C14, C16, C20: value 1uf -> 10uf
- U7: renamed from U10; value TL072 -> TL074; symbol Amplifier_Operational:TL072 -> Amplifier_Operational:TL074
- U8: renamed from U7; value TL072 -> TL074
- renumbered U4 to U1, U8 to U4, U9 to U5
Connections:
- net AB_BC: now also U5.6; no longer U5.2
- net EA_AB: now also U5.5; no longer U5.1
- net ExtL: now also U1.12; no longer U1.1
- net ExtR: now also U1.11; no longer U1.3
- net GND: now also U7.5 (+), U7.10 (+), U7.12 (+), U7.3 (+), U8.3 (+); no longer U7.3 (+)
- net XOR_SUM: now also U5.4; no longer U5.3
- net at C13.2, R40.2, R41.1: now also U7.7; no longer U7.1
- net at SW2.2 (B): now also U1.13; no longer U1.2
- net O_MIX2: now reaches R41.2
- net O_MIX2: now also R57.1
- new net: C13.1, R40.1, U6.5 (I_OUT2), U7.6 (-)
- new net: R56.2, R57.2, R58.2, R59.2, R60.1, U8.2 (-)
- new net: R60.2, R61.1, U8.1
- new net: C9.2, R50.2, R51.1, U7.1
- new net: C9.1, R50.1, U6.4 (I_OUT1), U7.2 (-)
- new net: C11.1, R54.1, U6.13 (I_OUT4), U7.13 (-)
- new net: C11.2, R54.2, R55.1, U7.14
- new net: C10.1, R52.1, U6.12 (I_OUT3), U7.9 (-)
- new net: C10.2, R52.2, R53.1, U7.8
- new net MAIN_OUT: R61.2
- new net O_MIX1: R51.2, R56.1
- new net O_MIX3: R53.2, R58.1
- new net O_MIX4: R55.2, R59.1
Other:
- note added: "TODO: add all ICs and caps"
- note added: "TODO: change diode circuit"
- moved on the sheet: C13, C14, C15, C16, C17, C18, C19, C20, C21, R13, R14, R15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
